File: build/icio500/icio500_clean.kicad_pcb (KiCad board)
At the start: 4 copper layers, 152.3 x 105 mm, 48 parts, among them J1 ?, U1 DC-DC ISO, U2 THAT1200, U3 TL072, U4 THAT1646, U5 Daisy Seed, U6 ?, U7 ?

Commit message: getting closer for daisy seed
Parts:
- moved C2 87.5 mm to (185.0, 145.0), turned to 90 degrees
- moved C4 83.2 mm to (185.0, 150.0), turned to 90 degrees
- moved U6 72.8 mm to (120.0, 145.0)
- moved C25 72.3 mm to (170.0, 93.0), turned to 90 degrees
- moved U7 65.0 mm to (125.0, 145.0)
- moved R7 62.6 mm to (160.0, 93.0), turned to 90 degrees
- moved D1 60.2 mm to (180.0, 145.0)
- moved C1 56.9 mm to (145.0, 126.0)
- moved C10 56.6 mm to (140.0, 118.0)
- moved C3 54.9 mm to (145.0, 134.0)
- moved R8 53.2 mm to (170.0, 87.0), turned to 90 degrees
- moved C11 48.1 mm to (140.0, 105.0)
- moved R1 48.0 mm to (146.0, 118.0)
- moved C18 46.7 mm to (173.0, 87.0)
- moved C26 46.1 mm to (153.0, 87.0), turned to 90 degrees
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Routing:
- net gnd: track 0.00 -> 277.4 mm, vias 0 -> 2
- net v_plus: track 0.00 -> 211.1 mm, vias 0 -> 6
- net v_minus: track 0.00 -> 159.1 mm, vias 0 -> 3
- net daisy_digital_gnd: track 0.00 -> 138.8 mm
- net chassis_gnd: track 0.00 -> 86.9 mm, vias 0 -> 2
- net out_plus_4dbu: track 0.00 -> 78.0 mm, vias 0 -> 3
- net daisy_audio_in: track 0.00 -> 75.9 mm, vias 0 -> 1
- net daisy_audio_out: track 0.00 -> 71.6 mm, vias 0 -> 1
- net out_minus: track 0.00 -> 68.2 mm, vias 0 -> 3
- net in_plus_4dbu: track 0.00 -> 62.8 mm, vias 0 -> 2
- net in_minus_4dbu: track 0.00 -> 60.4 mm, vias 0 -> 2
- net daisy_5v_power: track 0.00 -> 45.3 mm
- net daisy_d13: track 0.00 -> 42.3 mm
- net daisy_d14: track 0.00 -> 41.3 mm
- net audio_out_to_1646: track 0.00 -> 33.6 mm, vias 0 -> 3
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Other:
- board text removed: "BALANCED INPUT"
- board text removed: "DIGITAL PROCESSING"
- board text removed: "LINE DRIVER"
- board text removed: "POWER"
- board text removed: "SCALING"
