File: build/icio500/icio500.kicad_sch (KiCad schematic)
At the start: 1 part, among them J1 EDA 306

Commit message: daisy close to good
Parts:
- added C27, C28, C29: 220uF, Capacitor_SMD:CP_Elec_6.3x5.4, symbol Device:C_Polarized
Changed lines of the file:
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@@
 		)
 	)
+  (symbol (lib_id "Device:C_Polarized") (at 50 50 0) (unit 1)
+    (in_bom yes) (on_board yes) (dnp no) (fields_autoplaced yes)
+    (property "Reference" "C27" (at 53.81 48.73 0)
+      (effects (font (size 1.27 1.27)) (justify left))
+    )
+    (property "Value" "220uF" (at 53.81 51.27 0)
+      (effects (font (size 1.27 1.27)) (justify left))
+    )
+    (property "Footprint" "Capacitor_SMD:CP_Elec_6.3x5.4" (at 50 50 0)
+      (effects (font (size 1.27 1.27)) hide)
+    )
+    (property "Datasheet" "~" (at 50 50 0)
+      (effects (font (size 1.27 1.27)) hide)
+    )
+    (pin "1")
+    (pin "2")
+    (instances
+      (project "icio500"
+        (path "/d34350a0-ca36-45c2-a205-3160ab26ae70"
+          (reference "C27") (unit 1)
+        )
+      )
+    )
+  )
+  (global_label "daisy_5v_power" (shape input) (at 50 42.38 90) (fields_autoplaced yes)
+    (effects (font (size 1.27 1.27)) (justify left))
+    (property "Intersheetrefs" "${INTERSHEET_REFS}" (at 50 41.5 90)
+      (effects (font (size 1.27 1.27)) hide)
+    )
+  )
+  (global_label "gnd" (shape input) (at 50 57.62 270) (fields_autoplaced yes)
+    (effects (font (size 1.27 1.27)) (justify right))
+    (property "Intersheetrefs" "${INTERSHEET_REFS}" (at 50 58.5 270)
+      (effects (font (size 1.27 1.27)) hide)
+    )
+  )
+  (wire (pts (xy 50 46.19) (xy 50 42.38))
+    (stroke (width 0) (type default))
+  )
+  (wire (pts (xy 50 53.81) (xy 50 57.62))
+    (stroke (width 0) (type default))
+  )
+  (symbol (lib_id "Device:C_Polarized") (at 100 50 0) (unit 1)
+    (in_bom yes) (on_board yes) (dnp no) (fields_autoplaced yes)
+    (property "Reference" "C28" (at 103.81 48.73 0)
+      (effects (font (size 1.27 1.27)) (justify left))
+    )
+    (property "Value" "220uF" (at 103.81 51.27 0)
+      (effects (font (size 1.27 1.27)) (justify left))
+    )
+    (property "Footprint" "Capacitor_SMD:CP_Elec_6.3x5.4" (at 100 50 0)
+      (effects (font (size 1.27 1.27)) hide)
+    )
+    (property "Datasheet" "~" (at 100 50 0)
+      (effects (font (size 1.27 1.27)) hide)
+    )
+    (pin "1")
+    (pin "2")
+    (instances
+      (project "icio500"
+        (path "/5dabc73e-023a-4af6-a742-626472cd9aa4"
+          (reference "C28") (unit 1)
+        )
+      )
+    )
+  )
+  (global_label "v_plus" (shape input) (at 100 42.38 90) (fields_autoplaced yes)
+    (effects (font (size 1.27 1.27)) (justify left))
+    (property "Intersheetrefs" "${INTERSHEET_REFS}" (at 100 41.5 90)
+      (effects (font (size 1.27 1.27)) hide)
+    )
+  )
+  (global_label "gnd" (shape input) (at 100 57.62 270) (fields_autoplaced yes)
+    (effects (font (size 1.27 1.27)) (justify right))
+    (property "Intersheetrefs" "${INTERSHEET_REFS}" (at 100 58.5 270)
+      (effects (font (size 1.27 1.27)) hide)
+    )
+  )
+  (wire (pts (xy 100 46.19) (xy 100 42.38))
+    (stroke (width 0) (type default))
+  )
+  (wire (pts (xy 100 53.81) (xy 100 57.62))
+    (stroke (width 0) (type default))
+  )
+  (symbol (lib_id "Device:C_Polarized") (at 150 50 0) (unit 1)
+    (in_bom yes) (on_board yes) (dnp no) (fields_autoplaced yes)
+    (property "Reference" "C29" (at 153.81 48.73 0)
+      (effects (font (size 1.27 1.27)) (justify left))
+    )
+    (property "Value" "220uF" (at 153.81 51.27 0)
+      (effects (font (size 1.27 1.27)) (justify left))
+    )
+    (property "Footprint" "Capacitor_SMD:CP_Elec_6.3x5.4" (at 150 50 0)
+      (effects (font (size 1.27 1.27)) hide)
+    )
+    (property "Datasheet" "~" (at 150 50 0)
+      (effects (font (size 1.27 1.27)) hide)
+    )
+    (pin "1")
+    (pin "2")
+    (instances
+      (project "icio500"
+        (path "/3260f89a-1866-4df6-afab-e0bf0126dd52"
+          (reference "C29") (unit 1)
+        )
+      )
+    )
+  )
+  (global_label "v_minus" (shape input) (at 150 42.38 90) (fields_autoplaced yes)
+    (effects (font (size 1.27 1.27)) (justify left))
+    (property "Intersheetrefs" "${INTERSHEET_REFS}" (at 150 41.5 90)
+      (effects (font (size 1.27 1.27)) hide)
+    )
+  )
+  (global_label "gnd" (shape input) (at 150 57.62 270) (fields_autoplaced yes)
+    (effects (font (size 1.27 1.27)) (justify right))
+    (property "Intersheetrefs" "${INTERSHEET_REFS}" (at 150 58.5 270)
+      (effects (font (size 1.27 1.27)) hide)
+    )
+  )
+  (wire (pts (xy 150 46.19) (xy 150 42.38))
+    (stroke (width 0) (type default))
+  )
+  (wire (pts (xy 150 53.81) (xy 150 57.62))
+    (stroke (width 0) (type default))
+  )
 	(sheet_instances
 		(path "/"
