File: build/icio500/_autosave-icio500.kicad_pcb (KiCad board)
At the start: 4 copper layers, 152.3 x 105 mm, 58 parts, among them J1 ?, U1 ?, U2 ?, U3 ?, U4 ?, U5 ?, U6 ?

Commit message: footprints and placement getting closer
Parts:
- removed the U6 at (120.5, 135.2)
- removed edac 15: ?, Cards:EDA_306
