File: build/icio500/faceplate_logic.kicad_pcb (KiCad board)
At the start: 2 copper layers, 38.1 x 133.3 mm, 16 parts, among them U1 PinHeader_2x10_P2.54mm_Vertic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, U3 PinHeader_2x07_P2.54mm_Vertic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, U5 RotaryEncoder_Alps_EC11E-Swit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, U6 LED_0603_1608Metric, U7 LED_0603_1608Metric, U8 LED_0603_1608Metric, U9 LED_0603_1608Metric

Commit message: faceplate mockupo
Parts:
- removed U7, U8, U9: LED_0603_1608Metric, LED_0603_1608Metric
- added C10: , lib:C0402, F.Cu at (178.9, 117.9)
- added C11: , lib:C0402, F.Cu at (178.9, 114.9)
- added C12: , lib:C0603, F.Cu at (175.7, 118.9)
- added C13: , lib:C0603, F.Cu at (175.7, 112.9)
- added C14: , lib:C0603, F.Cu at (153.2, 113.9)
- added C15: , lib:C0603, F.Cu at (164.6, 89.9)
- added C16: , lib:C0603, F.Cu at (166.3, 97.4)
- added C17: , lib:C0603, F.Cu at (159.8, 91.6)
- added C18: , lib:C0603, F.Cu at (172.3, 91.7)
- added C19: , lib:C0402, F.Cu at (160.0, 78.0)
- added C20: , lib:C0402, F.Cu at (155.7, 78.0)
- added C21: ?, Capacitor_SMD:CP_Elec_5x5.4, F.Cu at (149.6, 76.4)
- added C22: ?, Capacitor_SMD:CP_Elec_5x5.4, F.Cu at (166.1, 76.2)
- added C23: , lib:C0603, F.Cu at (163.6, 72.0)
- added C24: , lib:C0603, F.Cu at (151.8, 72.1)
- added C25: ?, Capacitor_SMD:CP_Elec_6.3x5.4, F.Cu at (128.4, 136.5)
- added C26: ?, Capacitor_SMD:CP_Elec_6.3x5.4, F.Cu at (145.5, 89.3)
- added C27: ?, Capacitor_SMD:CP_Elec_6.3x5.4, F.Cu at (145.4, 98.2)
- added C3: ?, Capacitor_SMD:CP_Elec_6.3x5.4, F.Cu at (176.1, 145.1)
- added C4: , lib:C0603, F.Cu at (176.3, 140.1)
- added C5: , lib:C0603, F.Cu at (129.1, 131.3)
- added C6: , lib:C0603, F.Cu at (160.8, 140.1)
- added C7: , lib:C0603, F.Cu at (156.2, 119.4)
- added C8: , lib:C0603, F.Cu at (160.0, 111.4)
- added C9: , lib:C0402, F.Cu at (176.4, 116.4)
- added D1: ?, Diode_SMD:D_SMA, F.Cu at (176.3, 131.6)
- added D10: ?, Diode_SMD:D_SOD-123, F.Cu at (178.5, 76.2)
- added D2: ?, Diode_SMD:D_SMA, F.Cu at (176.3, 136.6)
- added D3: ?, Diode_SMD:D_SOD-123, F.Cu at (170.9, 114.4)
- added D4: ?, Diode_SMD:D_SOD-123, F.Cu at (170.9, 116.9)
- added D5: ?, Diode_SMD:D_SOD-123, F.Cu at (166.1, 114.4)
- added D6: ?, Diode_SMD:D_SOD-123, F.Cu at (166.1, 116.9)
- added D7: ?, Diode_SMD:D_SOD-123, F.Cu at (173.5, 71.2)
- added D8: ?, Diode_SMD:D_SOD-123, F.Cu at (173.5, 76.2)
- added D9: ?, Diode_SMD:D_SOD-123, F.Cu at (178.5, 71.2)
- added J1: ?, Cards:EDA_306, F.Cu at (198.5, 98.9)
- added R1: , lib:R0603, F.Cu at (178.9, 120.9)
- added R10: , lib:R0603, F.Cu at (151.9, 70.0)
- added R2: , lib:R0603, F.Cu at (179.1, 111.4)
- added U2: ?, Package_SO:SOIC-8_3.9x4.9mm_P1.27mm, F.Cu at (158.2, 115.4)
- added U4: ?, Package_SO:SOIC-8_3.9x4.9mm_P1.27mm, F.Cu at (157.8, 74.0)
- C1: value CP_Elec_6.3x5.4 -> ?; footprint CP_Elec_6.3x5.4 -> Capacitor_SMD:CP_Elec_6.3x5.4; moved to F.Cu
- C2: value CP_Elec_6.3x5.4 -> (none); footprint CP_Elec_6.3x5.4 -> lib:C0603; moved to F.Cu
- R3, R4, R5, R6, R7, R8, R9: value R_0603_1608Metric -> (none); footprint R_0603_1608Metric -> lib:R0603; moved to F.Cu
- U1: value PinHeader_2x10_P2.54mm_Vertical -> ?; footprint PinHeader_2x10_P2.54mm_Vertical -> Package_TO_SOT_THT:TO-220-3_Vertical; moved to F.Cu
- U3: value PinHeader_2x07_P2.54mm_Vertical -> ?; footprint PinHeader_2x07_P2.54mm_Vertical -> Package_SO:SOIC-8_3.9x4.9mm_P1.27mm
- U5: value RotaryEncoder_Alps_EC11E-Switch_Vertical_H20mm -> ?; footprint RotaryEncoder_Alps_EC11E-Switch_Vertical_H20mm -> Package_DIP:DIP-40_W15.24mm_Socket
- U6: value LED_0603_1608Metric -> ?; footprint LED_0603_1608Metric -> Connector_PinHeader_2.54mm:PinHeader_2x10_P2.54mm_Vertical
- moved R5 159.9 mm to (172.3, 89.5)
- moved R6 151.1 mm to (172.3, 93.8)
- moved R7 150.7 mm to (172.3, 97.9)
- moved C1 150.5 mm to (163.8, 135.1), turned to 180 degrees
- moved R8 149.4 mm to (172.3, 95.9)
- moved U1 149.0 mm to (165.8, 145.5), turned to 180 degrees
- moved R4 143.8 mm to (159.9, 93.7)
- moved U5 142.6 mm to (130.9, 112.5), turned to -90 degrees
- moved C2 141.5 mm to (166.3, 140.1), turned to 180 degrees
- moved R9 139.5 mm to (163.6, 70.0)
- moved R3 139.5 mm to (159.9, 95.8)
- moved U3 137.1 mm to (166.2, 93.7), turned to 0 degrees
- moved U6 98.6 mm to (93.4, 107.0), turned to 90 degrees
Connections:
- C1 pad 1: (no net) -> v_plus
- C1 pad 2: (no net) -> gnd
- C2 pad 1: (no net) -> v_plus
- C2 pad 2: (no net) -> gnd
- R3 pad 1: (no net) -> audio_out
- R3 pad 2: (no net) -> in_minus_1
- R4 pad 1: (no net) -> daisy_audio_in
- R4 pad 2: (no net) -> in_minus_1
- R5 pad 1: (no net) -> gnd
- R5 pad 2: (no net) -> in_minus_2
- R6 pad 1: (no net) -> audio_out_to_1646
- R6 pad 2: (no net) -> in_minus_2
- R7 pad 1: (no net) -> audio_in_from_daisy_plus
- R7 pad 2: (no net) -> in_plus_2
- R8 pad 1: (no net) -> gnd
- R8 pad 2: (no net) -> in_plus_2
- R9 pad 1: (no net) -> out_plus_4dbu
- R9 pad 2: (no net) -> driver.r_zobel_plus-vcc
- U1 pad 1: (no net) -> v_plus
- U1 pad 2: (no net) -> gnd
- U1 pad 3: (no net) -> daisy_5v_power
- U3 pad 1: (no net) -> daisy_audio_in
- U3 pad 2: (no net) -> in_minus_1
- U3 pad 3: (no net) -> gnd
- U3 pad 4: (no net) -> v_minus
- U3 pad 5: (no net) -> in_plus_2
- U3 pad 6: (no net) -> in_minus_2
- U3 pad 7: (no net) -> audio_out_to_1646
- U3 pad 8: (no net) -> v_plus
- U6 pad 1: (no net) -> daisy_5v_power
- U6 pad 2: (no net) -> audio_in_r
Routing:
- net v_plus: track 0.00 -> 180.6 mm, vias 0 -> 3
- net v_minus: track 0.00 -> 159.9 mm, vias 0 -> 2
- net daisy_5v_power: track 0.00 -> 113.1 mm
- net out_plus_4dbu: track 0.00 -> 74.5 mm, vias 0 -> 1
- net out_minus: track 0.00 -> 71.0 mm, vias 0 -> 1
- net audio_in_from_daisy_plus: track 0.00 -> 67.2 mm, vias 0 -> 1
- net daisy_audio_in: track 0.00 -> 60.7 mm, vias 0 -> 1
- net chassis_gnd: track 0.00 -> 58.0 mm, vias 0 -> 2
- net audio_in_r: track 0.00 -> 49.6 mm
- net gnd: track 0.00 -> 32.0 mm, vias 0 -> 22
- net v_minus_16v: track 0.00 -> 31.1 mm, vias 0 -> 1
- net v_plus_16v: track 0.00 -> 30.3 mm, vias 0 -> 1
- net in_plus_4dbu: track 0.00 -> 27.0 mm, vias 0 -> 1
- net audio_out_to_1646: track 0.00 -> 26.6 mm
- net in_minus_4dbu: track 0.00 -> 26.2 mm, vias 0 -> 1
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- added copper zone on B.Cu, net gnd
- added copper zone on F.Cu, net gnd
- added copper zone on In1.Cu, net gnd
Other:
- copper layers 2 -> 4
