File: build/icio500/faceplate_logic.kicad_sch (KiCad schematic)
At the start: 28 parts, among them J1 SM08B-SRSS-TB, U1 IS31FL3236

Commit message: idk
Parts:
- removed J1: SM08B-SRSS-TB, Connector_JST:JST_SH_SM08B-SRSS-TB_1x08-1MP_P1.00mm_Horizontal, symbol Local:JST_SH_8
- added J1: Conn_02x10, Connector_PinHeader_2.54mm:PinHeader_2x10_P2.54mm_Vertical, symbol Connector_Generic:Conn_02x10_Odd_Even
- C1, C2: symbol Local:C -> Device:C_Small
- D1, D10, D2, D3, D4, D5, D6, D7, D8, D9: symbol Local:LED -> Device:LED_Small
- ENC1: symbol Local:EC11E_Encoder -> Device:RotaryEncoder_Switch
- FB1: symbol Local:Ferrite_Bead -> Device:Ferrite_Bead_Small
- R1, R10, R11, R12, R2, R3, R4, R5, R6, R7, R8, R9: symbol Local:R -> Device:R_Small
- U1: symbol Local:IS31FL3236 -> Driver_LED:IS31FL3236-TQ
Changed lines of the file:
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@@
 		(company "ICIO")
 	)
-  (symbol
-    (lib_id "Local:JST_SH_8")
-    (at 30 50 0)
-    (unit 1) (exclude_from_sim no) (in_bom yes) (on_board yes)
-        (property "Reference" "J1"
-      (at 5 48 0)
-      (effects (font (size 1.27 1.27) (bold yes)) )
-    )
-        (property "Value" "SM08B-SRSS-TB"
-      (at 5 52 0)
-      (effects (font (size 1.27 1.27) ) )
-    )
-        (property "Footprint" "Connector_JST:JST_SH_SM08B-SRSS-TB_1x08-1MP_P1.00mm_Horizontal"
-      (at 0 0 0)
-      (effects (font (size 1.27 1.27) ) (hide yes))
-    )
-        (property "Datasheet" ""
-      (at 0 0 0)
-      (effects (font (size 1.27 1.27) ) (hide yes))
-    )
-  )
-  (symbol
-    (lib_id "Local:Ferrite_Bead")
+  (symbol (lib_id "Connector_Generic:Conn_02x10_Odd_Even") (at 30 50 0) (unit 1)
+    (in_bom yes) (on_board yes) (dnp no)
+    (property "Reference" "J1" (at 30 35 0)
+      (effects (font (size 1.27 1.27)))
+    )
+    (property "Value" "Conn_02x10" (at 30 37 0)
+      (effects (font (size 1.27 1.27)))
+    )
+    (property "Footprint" "Connector_PinHeader_2.54mm:PinHeader_2x10_P2.54mm_Vertical" (at 0 0 0)
+      (effects (font (size 1.27 1.27)) (hide yes))
+    )
+  )
+  (symbol
+    (lib_id "Device:Ferrite_Bead_Small")
     (at 55 35 0)
     (unit 1) (exclude_from_sim no) (in_bom yes) (on_board yes)
@@
   )
   (symbol
-    (lib_id "Local:C")
+    (lib_id "Device:C_Small")
     (at 68 35 0)
     (unit 1) (exclude_from_sim no) (in_bom yes) (on_board yes)
@@
   )
   (symbol
-    (lib_id "Local:C")
+    (lib_id "Device:C_Small")
     (at 78 35 0)
     (unit 1) (exclude_from_sim no) (in_bom yes) (on_board yes)
@@
   )
   (symbol
-    (lib_id "Local:R")
+    (lib_id "Device:R_Small")
     (at 88 25 0)
     (unit 1) (exclude_from_sim no) (in_bom yes) (on_board yes)
@@
   )
   (symbol
-    (lib_id "Local:R")
+    (lib_id "Device:R_Small")
     (at 98 25 0)
     (unit 1) (exclude_from_sim no) (in_bom yes) (on_board yes)
@@
   )
   (symbol
-    (lib_id "Local:IS31FL3236")
+    (lib_id "Driver_LED:IS31FL3236-TQ")
     (at 110 60 0)
     (unit 1) (exclude_from_sim no) (in_bom yes) (on_board yes)
@@
   )
   (symbol
-    (lib_id "Local:EC11E_Encoder")
+    (lib_id "Device:RotaryEncoder_Switch")
     (at 30 130 0)
     (unit 1) (exclude_from_sim no) (in_bom yes) (on_board yes)
@@
   )
   (symbol
-    (lib_id "Local:R")
+    (lib_id "Device:R_Small")
     (at 150 20 90)
     (unit 1) (exclude_from_sim no) (in_bom yes) (on_board yes)
@@
   )
   (symbol
-    (lib_id "Local:LED")
+    (lib_id "Device:LED_Small")
     (at 170 20 0)
     (unit 1) (exclude_from_sim no) (in_bom yes) (on_board yes)
@@
   )
   (symbol
-    (lib_id "Local:R")
+    (lib_id "Device:R_Small")
     (at 150 29 90)
     (unit 1) (exclude_from_sim no) (in_bom yes) (on_board yes)
@@
   )
   (symbol
-    (lib_id "Local:LED")
+    (lib_id "Device:LED_Small")
     (at 170 29 0)
     (unit 1) (exclude_from_sim no) (in_bom yes) (on_board yes)
@@
   )
   (symbol
-    (lib_id "Local:R")
+    (lib_id "Device:R_Small")
     (at 150 38 90)
     (unit 1) (exclude_from_sim no) (in_bom yes) (on_board yes)
@@
   )
   (symbol
-    (lib_id "Local:LED")
+    (lib_id "Device:LED_Small")
     (at 170 38 0)
     (unit 1) (exclude_from_sim no) (in_bom yes) (on_board yes)
@@
   )
   (symbol
-    (lib_id "Local:R")
+    (lib_id "Device:R_Small")
     (at 150 47 90)
     (unit 1) (exclude_from_sim no) (in_bom yes) (on_board yes)
@@
   )
   (symbol
-    (lib_id "Local:LED")
+    (lib_id "Device:LED_Small")
     (at 170 47 0)
     (unit 1) (exclude_from_sim no) (in_bom yes) (on_board yes)
@@
   )
   (symbol
-    (lib_id "Local:R")
+    (lib_id "Device:R_Small")
     (at 150 56 90)
     (unit 1) (exclude_from_sim no) (in_bom yes) (on_board yes)
@@
   )
   (symbol
-    (lib_id "Local:LED")
+    (lib_id "Device:LED_Small")
     (at 170 56 0)
     (unit 1) (exclude_from_sim no) (in_bom yes) (on_board yes)
@@
   )
   (symbol
-    (lib_id "Local:R")
+    (lib_id "Device:R_Small")
     (at 150 65 90)
     (unit 1) (exclude_from_sim no) (in_bom yes) (on_board yes)
@@
   )
   (symbol
-    (lib_id "Local:LED")
+    (lib_id "Device:LED_Small")
     (at 170 65 0)
     (unit 1) (exclude_from_sim no) (in_bom yes) (on_board yes)
@@
   )
   (symbol
-    (lib_id "Local:R")
+    (lib_id "Device:R_Small")
     (at 150 74 90)
     (unit 1) (exclude_from_sim no) (in_bom yes) (on_board yes)
@@
   )
   (symbol
-    (lib_id "Local:LED")
+    (lib_id "Device:LED_Small")
     (at 170 74 0)
     (unit 1) (exclude_from_sim no) (in_bom yes) (on_board yes)
@@
   )
   (symbol
-    (lib_id "Local:R")
+    (lib_id "Device:R_Small")
     (at 150 83 90)
     (unit 1) (exclude_from_sim no) (in_bom yes) (on_board yes)
@@
   )
   (symbol
-    (lib_id "Local:LED")
+    (lib_id "Device:LED_Small")
     (at 170 83 0)
     (unit 1) (exclude_from_sim no) (in_bom yes) (on_board yes)
@@
   )
   (symbol
-    (lib_id "Local:R")
+    (lib_id "Device:R_Small")
     (at 150 92 90)
     (unit 1) (exclude_from_sim no) (in_bom yes) (on_board yes)
@@
   )
   (symbol
-    (lib_id "Local:LED")
+    (lib_id "Device:LED_Small")
     (at 170 92 0)
     (unit 1) (exclude_from_sim no) (in_bom yes) (on_board yes)
@@
   )
   (symbol
-    (lib_id "Local:R")
+    (lib_id "Device:R_Small")
     (at 150 101 90)
     (unit 1) (exclude_from_sim no) (in_bom yes) (on_board yes)
@@
   )
   (symbol
-    (lib_id "Local:LED")
+    (lib_id "Device:LED_Small")
     (at 170 101 0)
     (unit 1) (exclude_from_sim no) (in_bom yes) (on_board yes)
@@
   (text "NOTE: ENC_A, ENC_B, ENC_SW route directly\nto Daisy GPIO via JST connector.\nDaisy handles quadrature decode in firmware." (at 15 145 0) (effects (font (size 1.5 1.5))))
   (text "I2C bus (SDA/SCL)\nIS31FL3236 addr: 0x3C (AD=GND)\n4.7k pull-ups to 3V3" (at 78 15 0) (effects (font (size 1.5 1.5))))
+  (global_label "+3V3" (shape input) (at 24.92 39.84 0) (fields_autoplaced yes) (property "Intersheet References" "" (at 0 0 0) (effects (font (size 1.27 1.27)) (hide yes))))
+  (global_label "+3V3" (shape input) (at 37.62 39.84 180) (fields_autoplaced yes) (property "Intersheet References" "" (at 0 0 0) (effects (font (size 1.27 1.27)) (hide yes))))
+  (global_label "GND" (shape input) (at 24.92 42.38 0) (fields_autoplaced yes) (property "Intersheet References" "" (at 0 0 0) (effects (font (size 1.27 1.27)) (hide yes))))
+  (global_label "SDA" (shape input) (at 37.62 42.38 180) (fields_autoplaced yes) (property "Intersheet References" "" (at 0 0 0) (effects (font (size 1.27 1.27)) (hide yes))))
+  (global_label "GND" (shape input) (at 24.92 44.92 0) (fields_autoplaced yes) (property "Intersheet References" "" (at 0 0 0) (effects (font (size 1.27 1.27)) (hide yes))))
+  (global_label "SCL" (shape input) (at 37.62 44.92 180) (fields_autoplaced yes) (property "Intersheet References" "" (at 0 0 0) (effects (font (size 1.27 1.27)) (hide yes))))
+  (global_label "GND" (shape input) (at 24.92 47.46 0) (fields_autoplaced yes) (property "Intersheet References" "" (at 0 0 0) (effects (font (size 1.27 1.27)) (hide yes))))
+  (global_label "ENC_A" (shape input) (at 37.62 47.46 180) (fields_autoplaced yes) (property "Intersheet References" "" (at 0 0 0) (effects (font (size 1.27 1.27)) (hide yes))))
+  (global_label "ENC_B" (shape input) (at 24.92 50 0) (fields_autoplaced yes) (property "Intersheet References" "" (at 0 0 0) (effects (font (size 1.27 1.27)) (hide yes))))
+  (global_label "ENC_SW" (shape input) (at 37.62 50 180) (fields_autoplaced yes) (property "Intersheet References" "" (at 0 0 0) (effects (font (size 1.27 1.27)) (hide yes))))
 )
