File: original_board.kicad_pcb (KiCad board)
At the start: 4 copper layers, 152.3 x 105 mm, 48 parts, among them J1 ?, U1 DC-DC ISO, U2 THAT1200, U3 TL072, U4 THAT1646, U5 Daisy Seed, U6 ?, U7 ?

Commit message: pretty ok layout for daisy
antigravity
Parts:
- removed C1, C3: ?, Capacitor_SMD:CP_Elec_6.3x5.4
- removed the C10 at (188.0, 98.0)
- removed the C11 at (188.0, 112.0)
- removed U1: DC-DC ISO, Converter_DCDC:Converter_DCDC_muRata_NMAxxxxSC_THT
- removed the U5 at (70.0, 105.0)
- removed U6, U7: ?, Connector_PinHeader_2.54mm:PinHeader_1x02_P2.54mm_Vertical
- J1: value ? -> EDA 306
- U3: renamed from U2; value THAT1200 -> ?
- U4: renamed from U3; value TL072 -> ?
- U5: renamed from U4; value THAT1646 -> ?
- moved D2 229.1 mm to (3.52, 10.2)
- moved D1 219.4 mm to (3.52, 16.8)
- moved U4 211.8 mm to (3.73, 2.73)
- moved R3 201.4 mm to (11.6, 14.6)
- moved R4 200.5 mm to (19.3, 9.21)
- moved R5 198.2 mm to (17.6, 19.1)
- moved R6 186.4 mm to (35.6, 19.1)
- moved C16 182.6 mm to (23.6, 23.6), turned to 0 degrees
- moved C13 176.0 mm to (17.6, 14.6), turned to 0 degrees
- moved C14 174.6 mm to (23.6, 19.1), turned to 0 degrees
- moved C15 168.6 mm to (29.6, 28.1), turned to 0 degrees
- moved C5 153.1 mm to (17.6, 32.6)
- moved C6 152.3 mm to (29.6, 23.6)
- moved C4 150.0 mm to (11.6, 32.6)
- moved C2 129.4 mm to (35.6, 23.6)
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- renumbered C12 to C10, C13 to C11, C14 to C12, C15 to C13, C16 to C14, C17 to C15, C18 to C16, C19 to C17, C20 to C18, C21 to C19, C22 to C20, C23 to C21, C24 to C22, C25 to C23, C26 to C24
Connections:
- net gain_trim renamed /GAIN_ADJ
- net in_minus_minus2dbu renamed /-IN-2
- net in_plus_minus2dbu renamed /+IN-2
- net out_plus_minus2dbu renamed /+OUT-2
- net stereo_link renamed /SC_LINK
- net v_minus_16v renamed -16V
- net v_plus_16v renamed +16V
- net v_plus_48v renamed +48V
- D3 pad 1: in_plus -> (no net)
- D3 pad 2: v_plus -> (no net)
- D4 pad 1: v_minus -> (no net)
- D4 pad 2: in_plus -> (no net)
- D5 pad 1: in_minus -> (no net)
- D5 pad 2: v_plus -> (no net)
- D6 pad 1: v_minus -> (no net)
- D6 pad 2: in_minus -> (no net)
- J1 pad 1: chassis_gnd -> /CHASSIS
- J1 pad 10: in_plus_4dbu -> /+IN+4
- J1 pad 13: gnd -> GND
- J1 pad 2: out_plus_4dbu -> /+OUT+4
- J1 pad 4: out_minus -> /-OUT
- J1 pad 5: gnd -> /AGND
- J1 pad 8: in_minus_4dbu -> /-IN+4
Other:
- copper layers 4 -> 2
- board text removed: "BALANCED INPUT"
- board text removed: "DIGITAL PROCESSING"
- board text removed: "LINE DRIVER"
- board text removed: "POWER"
- board text removed: "SCALING"
