File: commit_dfb5c8d.kicad_pcb (KiCad board)
At the start: 4 copper layers, 152.3 x 105 mm, 48 parts, among them J1 ?, U1 ?, U2 ?, U3 ?, U4 ?, U5 ?, U6 ?, U7 ?

Commit message: closer than ever
Parts:
- added C5: , lib:C0603, F.Cu at (150.1, 114.0)
- added C6: , lib:C0603, F.Cu at (150.1, 118.0)
- added U1: DC-DC ISO, Package_TO_SOT_THT:TO-220-3_Vertical, F.Cu at (154.3, 146.8)
- moved C15 42.7 mm to (145.5, 83.1)
- moved C16 42.7 mm to (134.5, 86.9)
- moved C17 42.7 mm to (134.5, 83.7)
- moved C18 42.7 mm to (145.5, 85.0)
- moved R3 42.7 mm to (132.0, 85.0)
- moved R4 42.7 mm to (132.0, 83.7)
- moved R5 42.7 mm to (148.0, 86.3)
- moved R6 42.7 mm to (148.0, 85.0)
- moved U3 42.7 mm to (140.0, 85.0)
- moved C5 20.2 mm to (90.9, 115.2)
- moved C6 20.2 mm to (96.9, 115.2)
- moved U5 20.2 mm to (50.0, 122.5)
- moved U6 20.2 mm to (70.0, 147.5)
- moved U7 20.2 mm to (90.0, 147.5)
- moved C19 20.0 mm to (172.5, 70.6)
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Routing:
- net gnd: track 0.00 -> 367.3 mm, vias 0 -> 7
- net v_plus: track 0.00 -> 136.0 mm, vias 0 -> 6
- net v_minus: track 0.00 -> 132.4 mm, vias 0 -> 4
- net daisy_audio_out: track 0.00 -> 111.9 mm, vias 0 -> 1
- net daisy_audio_in: track 0.00 -> 106.8 mm, vias 0 -> 1
- net audio_out_to_1646: track 0.00 -> 84.0 mm, vias 0 -> 2
- net chassis_gnd: track 0.00 -> 60.5 mm, vias 0 -> 2
- net audio_out: track 0.00 -> 55.0 mm, vias 0 -> 2
- net out_minus: track 0.00 -> 53.5 mm, vias 0 -> 1
- net out_plus_4dbu: track 0.00 -> 53.2 mm, vias 0 -> 1
- net in_plus_4dbu: track 0.00 -> 46.5 mm, vias 0 -> 2
- net in_minus_4dbu: track 0.00 -> 44.3 mm, vias 0 -> 2
- net daisy_d13: track 0.00 -> 31.4 mm
- net receiver.r_rf_plus-vcc: track 0.00 -> 28.3 mm, vias 0 -> 2
- net daisy_d14: track 0.00 -> 25.8 mm
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