File: commit_f17cf5f.kicad_pcb (KiCad board)
At the start: 4 copper layers, 152.3 x 105 mm, 48 parts, among them J1 ?, U1 ?, U2 ?, U3 ?, U4 ?, U5 ?, U6 ?, U7 ?

Commit message: closer than ever
Parts:
- U1: value ? -> DC-DC ISO; footprint Package_TO_SOT_THT:TO-220-3_Vertical -> Converter_DCDC:Converter_DCDC_muRata_NMAxxxxSC_THT
- U2: value ? -> THAT1200
- U3: value ? -> TL072
- U4: value ? -> THAT1646
- U5: value ? -> Daisy Seed
- moved R5 95.5 mm to (173.0, 141.3)
- moved C15 95.5 mm to (170.5, 138.1)
- moved C16 95.5 mm to (159.5, 141.9)
- moved C18 95.5 mm to (170.5, 140.0)
- moved R3 95.5 mm to (157.0, 140.0)
- moved R6 95.5 mm to (173.0, 140.0)
- moved U3 95.5 mm to (165.0, 140.0)
- moved C17 95.5 mm to (159.5, 138.7)
- moved R4 95.5 mm to (157.0, 138.7)
- moved C5 45.9 mm to (155.0, 100.0)
- moved C6 38.2 mm to (155.0, 110.0)
- moved C1 30.1 mm to (135.0, 100.0)
- moved C2 30.1 mm to (140.0, 100.0)
- moved C3 30.1 mm to (135.0, 110.0)
- moved C4 30.1 mm to (140.0, 110.0)
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Connections:
- C5 pad 2: gnd -> daisy_digital_gnd
- C6 pad 2: gnd -> daisy_digital_gnd
- D1 pad 1: v_plus -> (no net)
- D1 pad 2: v_plus_16v -> (no net)
- D2 pad 1: v_minus_16v -> (no net)
- D2 pad 2: v_minus -> (no net)
- D3 pad 1: v_plus -> in_plus
- D3 pad 2: in_plus -> v_plus
- D4 pad 1: in_plus -> v_minus
- D4 pad 2: v_minus -> in_plus
- D5 pad 1: v_plus -> in_minus
- D5 pad 2: in_minus -> v_plus
- D6 pad 1: in_minus -> v_minus
- D6 pad 2: v_minus -> in_minus
- U5 pad 40: gnd -> daisy_digital_gnd
- U6 pad 2: gnd -> daisy_digital_gnd
- U7 pad 2: gnd -> daisy_digital_gnd
Routing:
- net gnd: track 0.00 -> 271.1 mm, vias 0 -> 8
- net v_minus: track 0.00 -> 143.3 mm, vias 0 -> 5
- net v_plus: track 0.00 -> 139.4 mm, vias 0 -> 3
- net daisy_digital_gnd: track 0.00 -> 138.6 mm
- net daisy_audio_out: track 0.00 -> 118.2 mm, vias 0 -> 1
- net daisy_audio_in: track 0.00 -> 106.8 mm, vias 0 -> 1
- net daisy_5v_power: track 0.00 -> 97.4 mm, vias 0 -> 1
- net audio_out_to_1646: track 0.00 -> 80.2 mm, vias 0 -> 3
- net chassis_gnd: track 0.00 -> 60.2 mm, vias 0 -> 2
- net in_plus_4dbu: track 0.00 -> 54.3 mm, vias 0 -> 2
- net out_minus: track 0.00 -> 53.5 mm, vias 0 -> 1
- net audio_out: track 0.00 -> 52.7 mm, vias 0 -> 2
- net out_plus_4dbu: track 0.00 -> 48.9 mm, vias 0 -> 1
- net in_minus_4dbu: track 0.00 -> 44.9 mm, vias 0 -> 2
- net daisy_d13: track 0.00 -> 31.4 mm
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